File: hardware/PartiBadge-v2/PartiBadge-v2.brd (EAGLE design)
At the start: 119.8 x 118.6 mm, 30 parts, among them J1 I2C, J2 Supply

Commit message: revisions to brd v2
Parts:
- added IC1: (no value), v-reg:78XXS
- added PHOTON: PHOTON_WITH_HEADERS, Particle-Devices:PHOTON
- U$4: value PHOTON_WITH_HEADERS -> (none); device Particle-Devices:PHOTON -> particle-spark:SPARK-LOGO
- moved U$4 74.4 mm to (88.9, 63.5), flipped to the bottom, turned to 0 degrees
Connections:
- removed net 3V3: C1.1, J2.2, R10.2, R8.2, R9.2, SI7021.5, SJ1.2, U$2.BATTERY_POSITIVE, U$4.24, U$5.VCC
- removed net VIN: U$4.1
- new net +3V3: C1.1, IC1.OUT, J2.2, PHOTON.1, PHOTON.24, R10.2, R8.2, R9.2, SI7021.5, SJ1.2, U$5.VCC
- new net N$5: IC1.IN, U$2.BATTERY_POSITIVE
- net BUTTON_B: now also PHOTON.6; no longer U$4.6
- net BUTTON_G: now also PHOTON.5; no longer U$4.5
- net BUTTON_R: now also PHOTON.4; no longer U$4.4
- net BUTTON_Y: now also PHOTON.7; no longer U$4.7
- net CENT: now also PHOTON.16; no longer U$4.16
- net DOWN: now also PHOTON.19; no longer U$4.19
- net GND: now also IC1.GND, PHOTON.2, PHOTON.21; no longer U$4.2, U$4.21
- net IR_RECEIVER: now also PHOTON.12; no longer U$4.12
- net LED_B: now also PHOTON.10; no longer U$4.10
- net LED_G: now also PHOTON.9; no longer U$4.9
- net LED_R: now also PHOTON.8; no longer U$4.8
- net LED_Y: now also PHOTON.11; no longer U$4.11
- net LEFT: now also PHOTON.18; no longer U$4.18
- net N$1: now also PHOTON.3; no longer U$4.3
- net N$2: now also PHOTON.15; no longer U$4.15
- net RIGHT: now also PHOTON.17; no longer U$4.17
- net SCL: now also PHOTON.14; no longer U$4.14
- net SDA: now also PHOTON.13; no longer U$4.13
- net UP: now also PHOTON.20; no longer U$4.20
- net VBAT: now also PHOTON.22; no longer U$4.22
Routing:
- net +3V3: track 0.00 -> 239.3 mm, vias 0 -> 4
- net 3V3: track 211.2 -> 0.00 mm, vias 3 -> 0
- net N$5: track 0.00 -> 25.1 mm, vias 0 -> 1
- net GND: track 9.30 -> 33.4 mm
Other:
- board text added: "#BadgeLife"
- board text added: "3V3"
- board text added: "A"
- board text added: "B"
- board text added: "C"
- board text added: "D"
- board text added: "Display"
- board text added: "GND"
- board text added: "Game"
- board text added: "Particle.io"
- board text added: "SCL"
- board text added: "SDA"
- board text added: "particle.io"
